Commit message: Done script testing.

File: bullet_op3/data/models/robotis_op3.urdf (robot description, URDF)
Before this commit: robot robotis_op3, 23 links, 22 joints
Links:
- link body_link: geometry collision mesh filename=../meshes/body.stl scale=0.001 0.001 0.001; visual mesh filename=../meshes/body.stl scale=0.001 0.001 0.001
- link head_pan_link: geometry collision mesh filename=../meshes/h1.stl scale=0.001 0.001 0.001; visual mesh filename=../meshes/h1.stl scale=0.001 0.001 0.001
- link head_tilt_link: geometry collision mesh filename=../meshes/h2.stl scale=0.001 0.001 0.001; visual mesh filename=../meshes/h2.stl scale=0.001 0.001 0.001
- link l_ank_pitch_link: geometry collision mesh filename=../meshes/ll5.stl scale=0.001 0.001 0.001; visual mesh filename=../meshes/ll5.stl scale=0.001 0.001 0.001
- link l_ank_roll_link: geometry collision mesh filename=../meshes/ll6.stl scale=0.001 0.001 0.001; visual mesh filename=../meshes/ll6.stl scale=0.001 0.001 0.001
- link l_el_link: geometry collision mesh filename=../meshes/la3.stl scale=0.001 0.001 0.001; visual mesh filename=../meshes/la3.stl scale=0.001 0.001 0.001
- link l_hip_pitch_link: geometry collision mesh filename=../meshes/ll3.stl scale=0.001 0.001 0.001; visual mesh filename=../meshes/ll3.stl scale=0.001 0.001 0.001
- link l_hip_roll_link: geometry collision mesh filename=../meshes/ll2.stl scale=0.001 0.001 0.001; visual mesh filename=../meshes/ll2.stl scale=0.001 0.001 0.001
- link l_hip_yaw_link: geometry collision mesh filename=../meshes/ll1.stl scale=0.001 0.001 0.001; visual mesh filename=../meshes/ll1.stl scale=0.001 0.001 0.001
- link l_knee_link: geometry collision mesh filename=../meshes/ll4.stl scale=0.001 0.001 0.001; visual mesh filename=../meshes/ll4.stl scale=0.001 0.001 0.001
- link l_sho_pitch_link: geometry collision mesh filename=../meshes/la1.stl scale=0.001 0.001 0.001; visual mesh filename=../meshes/la1.stl scale=0.001 0.001 0.001
- link l_sho_roll_link: geometry collision mesh filename=../meshes/la2.stl scale=0.001 0.001 0.001; visual mesh filename=../meshes/la2.stl scale=0.001 0.001 0.001
- link r_ank_pitch_link: geometry collision mesh filename=../meshes/rl5.stl scale=0.001 0.001 0.001; visual mesh filename=../meshes/rl5.stl scale=0.001 0.001 0.001
- link r_ank_roll_link: geometry collision mesh filename=../meshes/rl6.stl scale=0.001 0.001 0.001; visual mesh filename=../meshes/rl6.stl scale=0.001 0.001 0.001
- link r_el_link: geometry collision mesh filename=../meshes/ra3.stl scale=0.001 0.001 0.001; visual mesh filename=../meshes/ra3.stl scale=0.001 0.001 0.001
- link r_hip_pitch_link: geometry collision mesh filename=../meshes/rl3.stl scale=0.001 0.001 0.001; visual mesh filename=../meshes/rl3.stl scale=0.001 0.001 0.001
- link r_hip_roll_link: geometry collision mesh filename=../meshes/rl2.stl scale=0.001 0.001 0.001; visual mesh filename=../meshes/rl2.stl scale=0.001 0.001 0.001
- link r_hip_yaw_link: geometry collision mesh filename=../meshes/rl1.stl scale=0.001 0.001 0.001; visual mesh filename=../meshes/rl1.stl scale=0.001 0.001 0.001
- link r_knee_link: geometry collision mesh filename=../meshes/rl4.stl scale=0.001 0.001 0.001; visual mesh filename=../meshes/rl4.stl scale=0.001 0.001 0.001
- link r_sho_pitch_link: geometry collision mesh filename=../meshes/ra1.stl scale=0.001 0.001 0.001; visual mesh filename=../meshes/ra1.stl scale=0.001 0.001 0.001
- link r_sho_roll_link: geometry collision mesh filename=../meshes/ra2.stl scale=0.001 0.001 0.001; visual mesh filename=../meshes/ra2.stl scale=0.001 0.001 0.001
